File: Tardis Board.sch (KiCad schematic (older format))
At the start: 17 parts, among them J1 Conn_01x03_Female, Q1 IRLB8721PBF, SW1 SW_DIP_x01, SW2 SW_DIP_x01, SW3 SW_DIP_x01, SW4 SW_DIP_x01, SW5 SW_DIP_x01, SW6 SW_DIP_x01, SW7 SW_DIP_x01

Commit message: Version 2 Ordered
Parts:
- removed SW2, SW3, SW4, SW5, SW6, SW7: SW_DIP_x01, Libraries:LED_CONNECTOR, symbol Switch:SW_DIP_x01
- added D2: 1N5817, Diode_THT:D_DO-41_SOD81_P10.16mm_Horizontal, symbol Diode:1N5817
- added SW2, SW3, SW4, SW5, SW6, SW7: SW_SPDT, Libraries:LED_CONNECTOR, symbol Switch:SW_SPDT
Connections:
- net labels added: 5v
- wire segments 103 -> 111
Other:
- moved on the sheet: SW1
